Commit message: feat: desviando perfeitamente do obstáculo e ajustando torques, usando 100% do potencial das 3 juntas

File: manipulador-planar/models/planar_arm_3dof.urdf (robot description, URDF)
Before this commit: robot planar_arm_3dof, 6 links, 5 joints
Joints:
- joint joint1: limit lower=-3.14 upper=3.14 effort=20 velocity=2.0 -> lower=-3.14 upper=3.14 effort=200 velocity=4.0
- joint joint2: limit lower=-3.14 upper=3.14 effort=20 velocity=2.0 -> lower=-3.14 upper=3.14 effort=200 velocity=4.0
- joint joint3: limit lower=-3.14 upper=3.14 effort=20 velocity=2.0 -> lower=-3.14 upper=3.14 effort=100 velocity=4.0
